Commit message: adding iCub3 with new arm cover

File: models/collisions_model/iCubGazeboV3_collisions/model.urdf (robot description, URDF)
Before this commit: robot iCub, 48 links, 47 joints
Links:
- link l_elbow_1: geometry visual mesh filename=package://iCub/meshes/simmechanics/sim_icub3_l_elbow_1_prt.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 scale=0.001 0.001 0.001
- link l_forearm: geometry visual mesh filename=package://iCub/meshes/simmechanics/sim_icub3_l_forearm_prt.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 scale=0.001 0.001 0.001
- link l_shoulder_1: geometry visual mesh filename=package://iCub/meshes/simmechanics/sim_icub3_l_shoulder_1_p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 scale=0.001 0.001 0.001
- link l_shoulder_2: geometry visual mesh filename=package://iCub/meshes/simmechanics/sim_icub3_l_shoulder_2_p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 scale=0.001 0.001 0.001
- link l_shoulder_3: geometry visual mesh filename=package://iCub/meshes/simmechanics/sim_icub3_l_shoulder_3_p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 scale=0.001 0.001 0.001
- link l_upper_arm: mass 2.06334 -> 2.07285
- link r_elbow_1: geometry visual mesh filename=package://iCub/meshes/simmechanics/sim_icub3_r_elbow_1_prt.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 scale=0.001 0.001 0.001
- link r_forearm: geometry visual mesh filename=package://iCub/meshes/simmechanics/sim_icub3_r_forearm_prt.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 scale=0.001 0.001 0.001
- link r_shoulder_1: geometry visual mesh filename=package://iCub/meshes/simmechanics/sim_icub3_r_shoulder_1_p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 scale=0.001 0.001 0.001
- link r_shoulder_2: geometry visual mesh filename=package://iCub/meshes/simmechanics/sim_icub3_r_shoulder_2_p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 scale=0.001 0.001 0.001
- link r_shoulder_3: geometry visual mesh filename=package://iCub/meshes/simmechanics/sim_icub3_r_shoulder_3_p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 scale=0.001 0.001 0.001
- link r_upper_arm: mass 2.06334 -> 2.07285; geometry collision mesh filename=package://iCub/meshes/simmechanics/sim_icub3_r_upperarm_ski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 scale=0.001 0.001 0.001; visual mesh filename=package://iCub/meshes/simmechanics/sim_icub3_r_upperarm_ski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 scale=0.001 0.001 0.001
Joints:
- joint chest_depth_frame_fixed_joint: origin xyz=0.0894115 0.0175 0.09929950000000001 rpy=-1.5707963267948968 0 -1.5707963267948968 -> xyz=0.0894115 0.0175 0.09929950000000001 rpy=-1.57079632679 0 -1.57079632679
- joint chest_rgb_frame_fixed_joint: origin xyz=0.0894115 -0.0115 0.09929950000000001 rpy=-1.5707963267948968 0 -1.5707963267948968 -> xyz=0.0894115 -0.0115 0.09929950000000001 rpy=-1.57079632679 0 -1.57079632679
- joint imu_frame_fixed_joint: origin xyz=0.0034999999997785457 0.0054999999863750895 0.1013340000004441 rpy=-3.141592653589793 0 -1.570796326794897 -> xyz=0.0034999999997785457 0.0054999999863750895 0.1013340000004441 rpy=-3.14159265359 0 -1.57079632679
- joint l_ankle_pitch: limit lower=-0.7853981633974483 upper=0.7853981633974483 effort=50000 velocity=120.0 -> lower=-0.785398163397 upper=0.785398163397 effort=50000 velocity=120.0
- joint l_ankle_roll: limit lower=-0.4363323129985824 upper=0.4363323129985824 effort=50000 velocity=120.0 -> lower=-0.436332312999 upper=0.436332312999 effort=50000 velocity=120.0
- joint l_arm_ft_sensor: origin xyz=-0.004350133156978329 3.632573233880443e-07 -0.05430003872406172 rpy=0 0 0 -> xyz=-0.004350133156978325 3.632573233880443e-07 -0.05430003872406172 rpy=0 0 0
- joint l_elbow: axis -8.811824154381087e-08 -1.0000002733514628 4.4047361189014644e-08 -> -8.811824153687198e-08 -1.0000002733514628 4.40473611855452e-08; limit lower=-0.05235987755982989 upper=1.3089969389957472 effort=50000 velocity=120.0 -> lower=-0.0523598775598 upper=1.308996939 effort=50000 velocity=120.0; origin xyz=0.009999930234919404 -0.001499647423428896 -0.12370033753758375 rpy=0 0 0 -> xyz=0.009999930234919404 -0.001499647423428896 -0.12370033753758373 rpy=0 0 0
- joint l_hip_pitch: limit lower=-0.7853981633974483 upper=2.007128639793479 effort=50000 velocity=120.0 -> lower=-0.785398163397 upper=2.00712863979 effort=50000 velocity=120.0
- joint l_hip_roll: limit lower=-0.17453292519943295 upper=2.007128639793479 effort=50000 velocity=120.0 -> lower=-0.174532925199 upper=2.00712863979 effort=50000 velocity=120.0
- joint l_hip_yaw: limit lower=-1.3962634015954636 upper=1.3962634015954636 effort=50000 velocity=120.0 -> lower=-1.3962634016 upper=1.3962634016 effort=50000 velocity=120.0
- joint l_knee: limit lower=-1.2217304763960306 upper=0.08726646259971647 effort=50000 velocity=120.0 -> lower=-1.2217304764 upper=0.0872664625997 effort=50000 velocity=120.0
- joint l_shoulder_pitch: axis 3.323079797673039e-07 0.9999999783534342 1.4452224303407313e-07 -> 3.323079797723505e-07 0.9999999783534342 1.4452224304101202e-07; limit lower=-1.53588974175501 upper=0.22689280275926285 effort=50000 velocity=120.0 -> lower=-1.53588974176 upper=0.226892802759 effort=50000 velocity=120.0; origin xyz=-0.020835100000000002 0.0397423 0.1052029 rpy=0.25326162380993705 -1.1977334179319483e-07 -0.26179930184968747 -> xyz=-0.020835100000000002 0.0397423 0.1052029 rpy=0.25326162381 -1.19773341793e-07 -0.26179930185
- joint l_shoulder_roll: axis 0.9999998262417684 2.0348252649342313e-07 -4.0230228454118944e-08 -> 0.9999998262417684 2.0348252649515786e-07 -4.0230228454118944e-08; limit lower=0.20943951023931956 upper=2.792526803190927 effort=50000 velocity=120.0 -> lower=0.157079632679 upper=2.84488668075 effort=50000 velocity=120.0; origin xyz=0.004992849331690818 0.111499838456099 0.0002686502277366859 rpy=-0.17453296140985 -0.05374759931933852 0 -> xyz=0.004992849331690818 0.111499838456099 0.0002686502277366859 rpy=-0.17453296141 -0.0537475993193 0
- joint l_shoulder_yaw: axis 2.227647404040578e-08 -4.393786245948661e-08 -1.0000002566182309 -> 2.227647404040578e-08 -4.393786245601716e-08 -1.0000002566182309; limit lower=-0.8726646259971648 upper=1.3962634015954636 effort=50000 velocity=120.0 -> lower=-0.872664625997 upper=1.3962634016 effort=50000 velocity=120.0; origin xyz=0 -4.2345248449371375e-07 -0.02249994137312443 rpy=0 0 0 -> xyz=0 -4.2345248449371375e-07 -0.022499941373124423 rpy=0 0 0
- joint l_wrist_pitch: axis -0.9999998262417684 -2.0348252649342313e-07 4.0230228454118944e-08 -> -0.9999998262417684 -2.0348252649515786e-07 4.0230228454118944e-08; limit lower=-1.2217304763960306 upper=0.4363323129985824 effort=50000 velocity=120.0 -> lower=-1.2217304764 upper=0.436332312999 effort=50000 velocity=120.0; origin xyz=0.016600015934286182 0.002006895218072541 -0.10749964114254112 rpy=0 0 0 -> xyz=0.016600015934286182 0.002006895218072541 -0.1074996411425411 rpy=0 0 0
- joint l_wrist_prosup: axis 2.227647404040578e-08 -4.393786245948661e-08 -1.0000002566182309 -> 2.227647404040578e-08 -4.393786245601716e-08 -1.0000002566182309; limit lower=-1.53588974175501 upper=1.53588974175501 effort=50000 velocity=120.0 -> lower=-1.53588974176 upper=1.53588974176 effort=50000 velocity=120.0; origin xyz=-0.014999870654177704 0.0019996435036348514 -0.055300063582479825 rpy=0 0 0 -> xyz=-0.0149998706541777 0.0019996435036348514 -0.055300063582479825 rpy=0 0 0
- joint l_wrist_yaw: axis 8.811824154381087e-08 1.0000002733514628 -4.4047361189014644e-08 -> 8.811824153687198e-08 1.0000002733514628 -4.40473611855452e-08; limit lower=-0.2617993877991494 upper=0.6108652381980153 effort=50000 velocity=120.0 -> lower=-0.261799387799 upper=0.610865238198 effort=50000 velocity=120.0; origin xyz=-0.016300121744729387 -0.0069993926815711816 0 rpy=0 0 0 -> xyz=-0.016300121744729383 -0.0069993926815711816 0 rpy=0 0 0
- joint neck_pitch: limit lower=-0.5235987755982988 upper=0.3839724354387525 effort=50000 velocity=120.0 -> lower=-0.523598775598 upper=0.383972435439 effort=50000 velocity=120.0
- joint neck_roll: limit lower=-0.3490658503988659 upper=0.3490658503988659 effort=50000 velocity=120.0 -> lower=-0.349065850399 upper=0.349065850399 effort=50000 velocity=120.0
- joint neck_yaw: limit lower=-0.7853981633974483 upper=0.7853981633974483 effort=50000 velocity=120.0 -> lower=-0.785398163397 upper=0.785398163397 effort=50000 velocity=120.0
- joint r_ankle_pitch: limit lower=-0.7853981633974483 upper=0.7853981633974483 effort=50000 velocity=120.0 -> lower=-0.785398163397 upper=0.785398163397 effort=50000 velocity=120.0
- joint r_ankle_roll: limit lower=-0.4363323129985824 upper=0.4363323129985824 effort=50000 velocity=120.0 -> lower=-0.436332312999 upper=0.436332312999 effort=50000 velocity=120.0
- joint r_arm_ft_sensor: origin xyz=-0.006849946385389875 2.1904996055921444e-07 -0.05429998157789099 rpy=0 0 0 -> xyz=-0.006849946385389879 2.1904996055921444e-07 -0.054299981577890996 rpy=0 0 0
- joint r_elbow: axis 2.4949582809984105e-07 -1.0000002733514362 2.7942487004772865e-08 -> 2.4949582810851467e-07 -1.0000002733514362 2.794248700824231e-08; limit lower=-0.05235987755982989 upper=1.3089969389957472 effort=50000 velocity=120.0 -> lower=-0.0523598775598 upper=1.308996939 effort=50000 velocity=120.0; origin xyz=0.009999931922603816 0.0014996401320274133 -0.1237003374895465 rpy=0 0 0 -> xyz=0.009999931922603813 0.0014996401320274133 -0.1237003374895465 rpy=0 0 0
- joint r_hip_pitch: limit lower=-0.7853981633974483 upper=2.007128639793479 effort=50000 velocity=120.0 -> lower=-0.785398163397 upper=2.00712863979 effort=50000 velocity=120.0
- joint r_hip_roll: limit lower=-0.17453292519943295 upper=2.007128639793479 effort=50000 velocity=120.0 -> lower=-0.174532925199 upper=2.00712863979 effort=50000 velocity=120.0
- joint r_hip_yaw: limit lower=-1.3962634015954636 upper=1.3962634015954636 effort=50000 velocity=120.0 -> lower=-1.3962634016 upper=1.3962634016 effort=50000 velocity=120.0
- joint r_knee: limit lower=-1.2217304763960306 upper=0.08726646259971647 effort=50000 velocity=120.0 -> lower=-1.2217304764 upper=0.0872664625997 effort=50000 velocity=120.0
- joint r_shoulder_pitch: axis 1.499044390054707e-07 0.9999999783534812 -1.2401537036188515e-07 -> 1.4990443900075867e-07 0.9999999783534812 -1.2401537036188515e-07; limit lower=-1.53588974175501 upper=0.22689280275926285 effort=50000 velocity=120.0 -> lower=-1.53588974176 upper=0.226892802759 effort=50000 velocity=120.0; origin xyz=-0.020835100000000002 -0.0397423 0.1052029 rpy=-0.25326164431680925 2.3014774394592079e-07 0.26179970938509745 -> xyz=-0.020835100000000002 -0.0397423 0.1052029 rpy=-0.253261644317 2.30147743946e-07 0.261799709385
- joint r_shoulder_roll: axis -0.9999998262417886 4.2105014356162707e-08 2.4630481189336084e-08 -> -0.9999998262417887 4.210501436396896e-08 2.463048118239719e-08; limit lower=0.20943951023931956 upper=2.792526803190927 effort=50000 velocity=120.0 -> lower=0.157079632679 upper=2.84488668075 effort=50000 velocity=120.0; origin xyz=0.007489008185044645 -0.11150041046657978 0.0004027858966975245 rpy=0.17453306234069357 -0.053747792579130614 -6.132332688812785e-07 -> xyz=0.007489008185044648 -0.11150041046657978 0.0004027858966975245 rpy=0.174533062341 -0.0537477925791 -6.13233268885e-07
- joint r_shoulder_yaw: axis -3.787621790513063e-08 2.805197706068352e-08 1.0000002566182309 -> -3.787621789819173e-08 2.8051977053744626e-08 1.0000002566182309; limit lower=-0.8726646259971648 upper=1.3962634015954636 effort=50000 velocity=120.0 -> lower=-0.872664625997 upper=1.3962634016 effort=50000 velocity=120.0
- joint r_wrist_pitch: axis 0.9999998262417886 -4.2105014356162707e-08 -2.4630481189336084e-08 -> 0.9999998262417887 -4.210501436396896e-08 -2.463048118239719e-08; limit lower=-1.2217304763960306 upper=0.4363323129985824 effort=50000 velocity=120.0 -> lower=-1.2217304764 upper=0.436332312999 effort=50000 velocity=120.0; origin xyz=0.016299953353948633 -0.002007442890811839 -0.10750007971210637 rpy=0 0 0 -> xyz=0.016299953353948637 -0.002007442890811839 -0.10750007971210643 rpy=0 0 0
- joint r_wrist_prosup: axis -3.787621790513063e-08 2.805197706068352e-08 1.0000002566182309 -> -3.787621789819173e-08 2.8051977053744626e-08 1.0000002566182309; limit lower=-1.53588974175501 upper=1.53588974175501 effort=50000 velocity=120.0 -> lower=-1.53588974176 upper=1.53588974176 effort=50000 velocity=120.0
- joint r_wrist_yaw: axis -2.4949582809984105e-07 1.0000002733514362 -2.7942487004772865e-08 -> -2.4949582810851467e-07 1.0000002733514362 -2.794248700824231e-08; origin xyz=-0.016300122874272734 0.0069993900510918194 0 rpy=0 0 0 -> xyz=-0.01630012287427273 0.0069993900510918194 0 rpy=0 0 0
- joint torso_pitch: limit lower=-0.3141592653589793 upper=0.7853981633974483 effort=50000 velocity=120.0 -> lower=-0.314159265359 upper=0.785398163397 effort=50000 velocity=120.0
- joint torso_roll: limit lower=-0.4014257279586958 upper=0.4014257279586958 effort=50000 velocity=120.0 -> lower=-0.401425727959 upper=0.401425727959 effort=50000 velocity=120.0
- joint torso_yaw: limit lower=-0.7504915783575618 upper=0.7504915783575618 effort=50000 velocity=120.0 -> lower=-0.750491578358 upper=0.750491578358 effort=50000 velocity=120.0

Commit message: updating model and meshes with most recent changes

File: models/collisions_model/iCubGazeboV3_collisions/model.urdf (robot description, URDF)
Before this commit: robot iCub, 48 links, 47 joints
Links:
- link r_upper_arm: geometry collision mesh filename=package://iCub/meshes/simmechanics/sim_icub3_r_upperarm_prt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 scale=0.001 0.001 0.001; visual mesh filename=package://iCub/meshes/simmechanics/sim_icub3_r_upperarm_prt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 scale=0.001 0.001 0.001
Joints:
- joint l_shoulder_roll: limit lower=0.157079632679 upper=2.84488668075 effort=50000 velocity=120.0 -> lower=0.157079632679 upper=2.87979326579 effort=50000 velocity=120.0; origin xyz=0.004992849331690818 0.111499838456099 0.0002686502277366859 rpy=-0.17453296141 -0.0537475993193 0 -> xyz=0.004992849331690818 0.111499838456099 0.0002686502277366859 rpy=-0.244346 -0.0537475993193 0
- joint r_shoulder_roll: limit lower=0.157079632679 upper=2.84488668075 effort=50000 velocity=120.0 -> lower=0.157079632679 upper=2.87979326579 effort=50000 velocity=120.0; origin xyz=0.007489008185044648 -0.11150041046657978 0.0004027858966975245 rpy=0.174533062341 -0.0537477925791 -6.13233268885e-07 -> xyz=0.007489008185044648 -0.11150041046657978 0.0004027858966975245 rpy=0.244346 -0.0537477925791 -6.13233268885e-07
